Commit message: update

File: catkin_ws/src/my_robot/urdf/my_robot.xacro (robot description, xacro)
@@ -8,4 +8,7 @@
     <child link="chassis" />
   </joint>
+ <gazebo reference="chassis">
+     <material>Gazebo/Blue</material>
+ </gazebo>
   <link name='chassis'>
     <pose>0 0 0.1 0 0 0</pose>
@@ -30,4 +33,7 @@
         <box size=".4 .2 .1"/>
       </geometry>
+      <material name="Blue">
+        <color rgba="0 0 1 1" />
+      </material>
     </visual>
     <collision name='back_caster_collision'>
@@ -56,4 +62,7 @@
     </visual>
   </link>
+ <gazebo reference="left_wheel">
+     <material>Gazebo/Green</material>
+ </gazebo>
   <link name='left_wheel'>
     <pose>0 0 0 0 0 0</pose>
@@ -79,5 +88,11 @@
       </geometry>
     </visual>
-  </link>
+      <material name="Green">
+        <color rgba="0 1 0 1" />
+      </material>
+  </link>
+ <gazebo reference="right_wheel">
+     <material>Gazebo/Green</material>
+ </gazebo>
   <link name='right_wheel'>
     <pose>0 0 0 0 0 0</pose>
@@ -102,4 +117,7 @@
         <cylinder radius="0.1" length="0.05"/>
       </geometry>
+      <material name="Green">
+        <color rgba="0 1 0 1" />
+      </material>
     </visual>
   </link>
@@ -120,4 +138,7 @@
     <dynamics damping="1.0" friction="1.0"/>
   </joint>
+ <gazebo reference="camera">
+     <material>Gazebo/Red</material>
+ </gazebo>
   <link name='camera'>
     <pose>0 0 0 0 0 0</pose>
@@ -142,4 +163,7 @@
         <box size="0.05 0.05 0.05"/>
       </geometry>
+      <material name="Red">
+        <color rgba="1 0 0 1" />
+      </material>
     </visual>
   </link>
